File: dam_connect/dam_connect.kicad_pcb (KiCad board)
At the start: 2 copper layers, 42.4 x 34.1 mm, 6 parts, among them J1 Conn_ARM_JTAG_SWD_20, J2 Conn_ARM_JTAG_SWD_10

Commit message: moved folder
Other:
- board text added: "JLCJLCJLCJLC"
Changed lines of the file:
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@@
 		(tags "Through hole horizontal IDC box header THT 2x10 2.54mm double row")
 		(property "Reference" "J1"
-			(at 8.9475 11.43 360)
+			(at 8.9475 11.43 0)
 			(layer "F.SilkS")
 			(effects
@@
 		)
 		(property "Value" "Conn_ARM_JTAG_SWD_20"
-			(at 23.1975 11.68 360)
+			(at 23.1975 11.68 0)
 			(layer "F.Fab")
 			(effects
@@
 		)
 		(property "Value" "SolderJumper_3_Bridged12"
-			(at -4.75 -2 360)
+			(at -4.75 -2 0)
 			(layer "F.Fab")
 			(effects
@@
 		)
 		(fp_text user "3"
-			(at 2.6 0 360)
+			(at 2.6 0 0)
 			(layer "F.SilkS")
 			(effects
@@
 		)
 		(fp_text user "1"
-			(at -2.6 0 360)
+			(at -2.6 0 0)
 			(layer "F.SilkS")
 			(effects
@@
 		(fill none)
 		(layer "Edge.Cuts")
+	)
+	(gr_text "JLCJLCJLCJLC"
+		(at 178 84 90)
+		(layer "B.SilkS")
+		(effects
+			(font
+				(size 1 1)
+				(thickness 0.2)
+				(bold yes)
+			)
+			(justify left bottom mirror)
+		)
 	)
 	(gr_text "AD PW"
@@
 			(thermal_gap 0.5)
 			(thermal_bridge_width 0.5)
-			(smoothing fillet)
 		)
 		(polygon
@@
 			(thermal_gap 0.5)
 			(thermal_bridge_width 0.5)
-			(smoothing fillet)
 		)
 		(polygon
@@
 			(thermal_gap 0.5)
 			(thermal_bridge_width 0.5)
-			(smoothing fillet)
 		)
 		(polygon
@@
 			(thermal_gap 0.5)
 			(thermal_bridge_width 0.5)
-			(smoothing fillet)
 		)
 		(polygon
