File: DAMLink.kicad_pcb (KiCad board)
At the start: 2 copper layers, 41 x 33 mm, 75 parts, among them J1 PicoBlade, J2 USB_C_Receptacle_Host, J3 PicoBlade, J4 VCCIO_EXT, J5 TC2050-IDC, J6 Conn_ST_STDC14, P1 USB_C_Plug, SW1 SW_DIP_x04, U1 FT230XQ, U2 USB3740B-AI2, U3 TMUX1574RSVR, U4 USBLC6-4SC6, U5 SiP32432DR3, U6 USBLC6-4SC6

Commit message: pushed schematics to pcb
Parts:
- added JP102: SolderJumper_2_Open, Jumper:SolderJumper-2_P1.3mm_Open_TrianglePad1.0x1.5mm, F.Cu at (103.0, 40.2)
- added JP103: SolderJumper_2_Open, Jumper:SolderJumper-2_P1.3mm_Open_TrianglePad1.0x1.5mm, F.Cu at (103.0, 43.8)
- moved U103 108.6 mm to (177.2, 49.8), turned to 180 degrees
- moved U101 96.7 mm to (170.7, 52.7)
- moved U105 96.3 mm to (163.8, 47.8)
- moved J101 95.7 mm to (169.1, 43.7), turned to 180 degrees
- moved J105 90.7 mm to (177.8, 66.6)
- moved J106 88.3 mm to (176.9, 42.5)
- moved U104 85.1 mm to (181.9, 48.4)
- moved U106 85.1 mm to (181.9, 53.0)
- moved U102 77.7 mm to (161.8, 52.0)
- moved SW101 72.8 mm to (160.9, 60.7)
- moved JP104 43.8 mm to (137.9, 31.6)
- moved TP103 43.8 mm to (124.0, 35.0)
- moved TP106 43.8 mm to (123.5, 32.6)
- moved TP107 43.8 mm to (127.8, 30.9)
- moved TP112 43.8 mm to (117.0, 36.9)
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- renumbered C1 to C101, C2 to C102, C3 to C103, C4 to C104, C5 to C105, D1 to D101, D2 to D102, D3 to D103, FB1 to FB101, H1 to H101, H2 to H102, H3 to H103, H4 to H104, J1 to J101, J2 to J102, J3 to J103, J4 to J104, J5 to J105, J6 to J106, JP1 to JP101, JP2 to JP104, JP3 to JP105, JP4 to JP106, JP5 to JP107, JP6 to JP108, JP7 to JP109, P1 to P101, R1 to R101, R2 to R102, R3 to R103, R4 to R104, R5 to R105, R6 to R106, R7 to R107, R8 to R108, R9 to R109, R10 to R110, R11 to R111, R12 to R112, R13 to R113, R14 to R114, SW1 to SW101, TP1 to TP101, TP2 to TP102, TP3 to TP103, TP4 to TP104, TP5 to TP105, TP6 to TP106, TP7 to TP107, TP8 to TP108, TP9 to TP109, TP10 to TP110, TP11 to TP111, TP12 to TP112, TP13 to TP113, TP14 to TP114, TP15 to TP115, TP16 to TP116, TP17 to TP117, U1 to U101, U2 to U102, U3 to U103, U4 to U104, U5 to U105, U6 to U106
Connections:
- U101 pad 15: Net-(JP8-A) -> Net-(JP102-A)
- U101 pad 2: Net-(JP9-A) -> Net-(JP103-A)

Commit message: Working on PCB
Parts:
- moved FB101 84.5 mm to (158.3, 57.2)
- moved R101 79.3 mm to (153.2, 56.8), turned to 180 degrees
- moved R102 79.2 mm to (157.1, 43.8), turned to 180 degrees
- moved C101 65.8 mm to (139.4, 46.8)
- moved C102 65.8 mm to (139.4, 49.3)
- moved C104 65.8 mm to (139.4, 54.3)
- moved J106 26.1 mm to (167.0, 66.6)
- moved U101 18.7 mm to (156.7, 40.3), turned to 90 degrees
- moved SW101 7.02 mm to (157.8, 67.0)
- moved U106 4.81 mm to (182.8, 48.3)
- moved U104 3.71 mm to (182.8, 52.0)
- moved U102 2.52 mm to (163.9, 50.6), turned to 135 degrees
- turned U103 to 0 degrees
Routing:
- net /SWT_RX-: track 0.00 -> 43.6 mm
- net /~{RESET}: track 0.00 -> 36.7 mm
- net /VBUS_DEV: track 0.00 -> 32.7 mm
- net /DEV_D-: track 0.00 -> 30.4 mm
- net /SWO: track 0.00 -> 28.2 mm
- net /DEV_D+: track 0.00 -> 25.3 mm, vias 0 -> 2
- net /SWCLK: track 0.00 -> 21.8 mm
- net /UART_USB: track 0.00 -> 19.8 mm, vias 0 -> 2
- net /SWDIO: track 0.00 -> 19.0 mm
- net /DEV_RX+: track 0.00 -> 14.6 mm
- net /UART_D-: track 0.00 -> 13.1 mm
- net /UART_D+: track 0.00 -> 12.4 mm
- net /HOST_D-: track 0.00 -> 11.7 mm, vias 0 -> 2
- net /HOST_D+: track 0.00 -> 9.64 mm, vias 0 -> 2
- net /DEV_RX-: track 0.00 -> 9.44 mm
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
Commit message: add new pcb file
Add new pcb file since the old one has some strange artefacts.
Parts:
- removed C101: 10nF, Capacitor_SMD:C_0603_1608Metric
- removed C102, C103, C105: 100nF, Capacitor_SMD:C_0603_1608Metric
- removed C104: 1uF, Capacitor_SMD:C_0603_1608Metric
- removed D101: TXD, LED_SMD:LED_0603_1608Metric
- removed D102: RXD, LED_SMD:LED_0603_1608Metric
- removed D103: WHITE, LED_SMD:LED_0603_1608Metric
- removed FB101: 120R/0.55A, Inductor_SMD:L_0603_1608Metric
- removed G***: LOGO, LOGO
- removed H101, H102, H103, H104: MountingHole_Pad, MountingHole:MountingHole_2.7mm_M2.5_ISO7380_Pad
- removed J101: PicoBlade, Connector_Molex:Molex_PicoBlade_53048-0610_1x06_P1.25mm_Horizontal
- removed J102: USB_C_Receptacle_Host, Connector_USB:USB_C_Receptacle_Amphenol_12401610E4-2A
- removed J103: PicoBlade, Connector_PinHeader_1.27mm:PinHeader_1x04_P1.27mm_Vertical
- removed J104: VCCIO_EXT, Connector_PinHeader_1.27mm:PinHeader_1x02_P1.27mm_Vertical
- removed J105: TC2050-IDC, Connector:Tag-Connect_TC2050-IDC-FP_2x05_P1.27mm_Vertical
- removed J106: Conn_ST_STDC14, Connector_STDC14:CON14_2X7_DUK_FTSH_SAI
- removed JP101, JP108, JP109, JP8, JP9: SolderJumper_2_Bridged, Jumper:SolderJumper-2_P1.3mm_Bridged_RoundedPad1.0x1.5mm
- removed JP102, JP103: SolderJumper_2_Open, Jumper:SolderJumper-2_P1.3mm_Open_TrianglePad1.0x1.5mm
- removed JP104 (x2), JP105 (x2), JP107: SolderJumper_3_Bridged12, Jumper:SolderJumper-3_P1.3mm_Bridged12_RoundedPad1.0x1.5mm
- removed JP106: SolderJumper_2_Open, Jumper:SolderJumper-2_P1.3mm_Open_RoundedPad1.0x1.5mm
- removed P101: USB_C_Plug, Connector_USB:USB_C_Plug_Molex_105444
- removed R101, R102: 5k1, Resistor_SMD:R_0603_1608Metric
- removed R103, R104, R111: 22k, Resistor_SMD:R_0603_1608Metric
- removed R105, R106, R112: 1k, Resistor_SMD:R_0603_1608Metric
- removed R107, R108, R109, R110: 680R, Resistor_SMD:R_0603_1608Metric
- removed R113: 22k, Resistor_SMD:R_0603_1608Metric_Pad0.98x0.95mm_HandSolder
- removed R114: 10k, Resistor_SMD:R_0603_1608Metric_Pad0.98x0.95mm_HandSolder
- removed SW101: SW_DIP_x04, Button_Switch_SMD:SW_DIP_SPSTx04_Slide_Copal_CHS-04A_W5.08mm_P1.27mm_JPin
- removed TP101, TP102, TP103, TP104, TP105, TP106, TP107, TP108, TP109, TP110, TP111, TP112, TP113 (x2), TP114 (x2), TP115 (x2), TP116 (x2), TP117 (x2): TestPoint_Small, TestPoint:TestPoint_Pad_D1.0mm
- removed U101: FT230XQ, Package_DFN_QFN:QFN-16-1EP_4x4mm_P0.65mm_EP2.1x2.1mm
- removed U102: USB3740B-AI2, Package_DFN_QFN:UQFN-10_1.3x1.8mm_P0.4mm
- removed U103: TMUX1574RSVR, TMUX1574RSVR:RSV16_TEX
- removed U104, U106: USBLC6-4SC6, Package_TO_SOT_SMD:SOT-23-6
- removed U105: SiP32432DR3, Package_TO_SOT_SMD:SOT-363_SC-70-6
Routing:
- net /SWT_RX-: track 43.6 -> 0.00 mm
- net /~{RESET}: track 36.7 -> 0.00 mm
- net /VBUS_DEV: track 32.7 -> 0.00 mm
- net /DEV_D-: track 30.4 -> 0.00 mm
- net /SWO: track 28.2 -> 0.00 mm
- net /DEV_D+: track 25.3 -> 0.00 mm, vias 2 -> 0
- net /SWCLK: track 21.8 -> 0.00 mm
- net /UART_USB: track 19.8 -> 0.00 mm, vias 2 -> 0
- net /SWDIO: track 19.0 -> 0.00 mm
- net /DEV_RX+: track 14.6 -> 0.00 mm
- net /UART_D-: track 13.1 -> 0.00 mm
- net /UART_D+: track 12.4 -> 0.00 mm
- net /HOST_D-: track 11.7 -> 0.00 mm, vias 2 -> 0
- net /HOST_D+: track 9.64 -> 0.00 mm, vias 2 -> 0
- net /DEV_RX-: track 9.44 -> 0.00 mm
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Other:
- board outline removed
- copper layers 2 -> 6
- board text removed: "3V3"
- board text removed: "ARM-JTAG/SWD"
- board text removed: "CB0"
- board text removed: "CB1"
- board text removed: "CB2"
- board text removed: "CB3"
- board text removed: "DAMLink R${REVISION}"
- board text removed: "DEVICE"
- board text removed: "DEV_D+"
- board text removed: "DEV_D-"
- board text removed: "DEV_RX+"
- board text removed: "DEV_RX-"
- board text removed: "GND"
- board text removed: "HOST"
- board text removed: "HOST_D+"
- board text removed: "HOST_D-"
- board text removed: "NRST"
- board text removed: "RXD"
- board text removed: "SWCLK"
- board text removed: "SWDIO"
- board text removed: "SWO"
- board text removed: "TC-2030"
- board text removed: "TXD"
- board text removed: "UART_D+"
- board text removed: "UART_D-"
- board text removed: "UART_USB"
- board text removed: "URXD->DEV_RXD"
- board text removed: "USB-C DAM Tool"
- board text removed: "UTXD<-DEV_TXD"
- board text removed: "VBUS->VBDEV"
- board text removed: "VCC"
- board text removed: "VCCIO"
- board text removed: "VEXT"
- board text removed: "VTGT"
- board text removed: "VTRG"
- board text removed: "~{PASS_USB}"
